File: corne-classic/pcb/corne-classic.sch (KiCad schematic (older format))
At the start: 87 parts, among them J1 MJ-4PP-9, J2 OLED, J3 LED, P1 i2c-pin, P2 i2c-pin, SW1 SW_PUSH, SW10 SW_PUSH, SW11 SW_PUSH, SW12 SW_PUSH, SW13 SW_PUSH, SW14 SW_PUSH, SW15 SW_PUSH, SW16 SW_PUSH, SW17 SW_PUSH, SW18 SW_PUSH, SW19 SW_PUSH, SW2 SW_PUSH, SW20 SW_PUSH, SW21 SW_PUSH, SW3 SW_PUSH, SW4 SW_PUSH, SW5 SW_PUSH, SW6 SW_PUSH, SW7 SW_PUSH, SW8 SW_PUSH, SW9 SW_PUSH, U1 ProMicro

Commit message: Adding one layer of keys
Parts:
- added D22, D23, D24, D25, D26, D27: D, kbd:D3_TH_SMD, symbol Device:D
- added L28, L29, L30, L31, L32, L33: SK6812MINI, kbd:SK6812MINI_rev, symbol corne-classic-rescue:SK6812MINI-kbd
- added SW22, SW23, SW24, SW25, SW26, SW27: SW_PUSH, kbd:MX_ALPS_PG1350_noLed, symbol corne-classic-rescue:SW_PUSH-kbd
- J1: symbol kbd:MJ-4PP-9 -> corne-classic-rescue:MJ-4PP-9-kbd
- L1, L10, L11, L12, L13, L14, L15, L16, L17, L18, L19, L2, L20, L21, L22, L23, L24, L25, L26, L27, L3, L4, L5, L6, L7, L8, L9: symbol kbd:SK6812MINI -> corne-classic-rescue:SK6812MINI-kbd
- RSW1, SW1, SW10, SW11, SW12, SW13, SW14, SW15, SW16, SW17, SW18, SW19, SW2, SW20, SW21, SW3, SW4, SW5, SW6, SW7, SW8, SW9: symbol kbd:SW_PUSH -> corne-classic-rescue:SW_PUSH-kbd
- U1: symbol kbd:ProMicro -> corne-classic-rescue:ProMicro-kbd
Connections:
- net labels added: row4
- wire segments 265 -> 326
- no-connect marks 6 -> 5
Other:
- moved on the sheet: D1, D10, D11, D12, D13, D14, D15, D16, D17, D18, D19, D2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
